Commit message: arbrob_v0.1 - working xacro

File: docker/moveit-arbrob/src/arbrob/urdf/print_tool.xacro (robot description, xacro)
@@ -9,5 +9,5 @@
       <child link="${prefix}print_tool"/>
       <!-- The tool is directly attached to the flange. -->
-      <origin rpy="0 0 0" xyz="0 0 0"/>
+      <origin rpy="0 0 ${pi/-2}" xyz="0 0 0"/>
     </joint>
     <link name="${prefix}print_tool">
@@ -24,10 +24,15 @@
         </geometry>
       </collision>
+      <inertial>
+        <origin rpy="0 0 0" xyz="0.03000526 0.00000117 0.02086005"/>
+        <mass value="0.4" />
+        <inertia ixx="1.72041901e-08" ixy="1.0914e-12" ixz="-1.2969622799999999e-08" iyy="1.0914e-12" iyz="4.3562402300000004e-08" izz="-4.2000000000000004e-14"/>
+      </inertial>
     </link>
     <!-- TCP frame -->
-    <joint name="${prefix}tcp_joint" type="revolute">
-      <axis xyz="0 0 1"/>
-      <limit effort="1000.0" lower="0.0" upper="0.78539816339745" velocity="0.5"/>
-      <origin xyz="0.08 0 0.022" rpy="0 0 0"/>
+    <joint name="${prefix}tcp_joint" type="fixed">
+      <!--axis xyz="0 0 1"/ -->
+      <origin xyz="0.08 0 0.022" rpy="${pi/2} 0 ${pi/-2}"/>
+      <!-- limit effort="1000.0" lower="-0.5" upper="0.5" velocity="0.5"/ -->
       <parent link="${prefix}print_tool"/>
       <child link="${prefix}tcp"/>

File: docker/moveit-arbrob/src/arbrob/urdf/ur5_rack_with_print_tool.urdf (robot description, URDF)
Before this commit: robot ur5_with_print_tool, 13 links, 12 joints
Links:
- added link U0CF
- added link axisA; collision mesh filename=package://arbrob/meshes/servo/collision/servo_head_v0.1.stl; visual mesh filename=package://arbrob/meshes/servo/visual/servo_head_v0.1.stl
- added link rack; collision mesh filename=package://arbrob/meshes/rack/collision/rack_v0.1.stl; visual mesh filename=package://arbrob/meshes/rack/visual/rack_v0.1.stl
- added link servo; collision mesh filename=package://arbrob/meshes/servo/collision/servo_body_v0.1.stl; visual mesh filename=package://arbrob/meshes/servo/visual/servo_body_v0.1.stl
- added link servo_link
- added link ur_link
- link print_tool: mass None -> 0.4
Joints:
- added joint attachment_U0CF: type fixed, parent axisA, child U0CF, origin xyz=0.0 0.0 0.0 rpy=1.57079632679 -1.57079632679 0.0
- added joint attachment_UR5: type fixed, parent rack, child ur_link, origin xyz=0.54 0.119 0.428 rpy=0.0 0.0 0.0
- added joint attachment_joint_ur: type fixed, parent ur_link, child base_link, origin xyz=0.0 0.0 0.0 rpy=0.0 0.0 0.0
- added joint attachment_servo: type fixed, parent rack, child servo_link, origin xyz=0.02 0.65 0.44 rpy=0.0 0.0 0.0
- added joint axisA_joint: type continuous, parent servo, child axisA, origin xyz=0.0155 0.0 0.0352 rpy=-1.57079632679 0.0 -1.57079632679, axis 0 0 1
- added joint servo_joint: type fixed, parent servo_link, child servo, origin xyz=0 0 0 rpy=0 0 0
- joint print_tool_joint: origin xyz=0 0 0 rpy=0 0 0 -> xyz=0 0 0 rpy=0 0 -1.57079632679
- joint tcp_joint: axis 0 0 1 -> (none); limit lower=0.0 upper=0.78539816339745 effort=1000.0 velocity=0.5 -> (none); origin xyz=0.08 0 0.022 rpy=0 0 0 -> xyz=0.08 0 0.022 rpy=1.57079632679 0 -1.57079632679; type revolute -> fixed
- joint world_joint: child base_link -> rack

File: docker/moveit-arbrob/src/arbrob/urdf/ur5_rack_with_print_tool.xacro (robot description, xacro)
@@ -1,4 +1,8 @@
 <?xml version="1.0"?>
-<robot name="ur5_with_print_tool" xmlns:xacro="http://wiki.ros.org/xacro">
+<robot name="ur5_rack_with_print_tool" xmlns:xacro="http://wiki.ros.org/xacro">
+  <!-- rack -->
+  <xacro:include filename="rack.xacro"/>
+  <!-- servo -->
+  <xacro:include filename="servo.xacro"/>
   <!-- ur5 -->
   <xacro:include filename="$(find ur_description)/urdf/ur5.urdf.xacro" />
@@ -8,14 +12,19 @@
   <!-- The ur5 xacro must be included with passing parameters -->
   <xacro:ur5_robot prefix="" joint_limited="true"/>
-  <!-- end-effector -->
   <!-- Here we include the end-effector by setting the parameters -->
   <!-- TODO: check end-effector link name of robot -->
   <xacro:print_tool prefix="" connected_to="tool0"/>
-  <!-- define the ur5's position and orientation in the world coordinate system -->
   <link name="world" />
   <joint name="world_joint" type="fixed">
     <parent link="world" />
-    <child link="base_link" /> <!-- TODO: check base_link name of robot -->
+    <child link="rack" />
     <origin xyz="0.0 0.0 0.0" rpy="0.0 0.0 0.0" />
   </joint>
+  <xacro:rack prefix=""/>
+  <joint name="attachment_joint_ur" type="fixed">
+    <parent link="ur_link" />
+    <child link="base_link" />
+    <origin xyz="0.0 0.0 0.0" rpy="0.0 0.0 0.0" />
+  </joint>
+  <xacro:servo prefix="" connected_to="servo_link"/>
 </robot>
